File: PS-MotorControllerInterfacePCB.kicad_pcb (KiCad board)
At the start: 2 copper layers, 59.1 x 75.7 mm, 124 parts, among them IC1 LM74502HDDFR, IC2 LM74502HDDFR, J1 53307-2471, J2 MotorController-in, J3 Conn_01x06, J4 PEAK, J5 Power MPPT, J6 MotorController-out, J7 Conn_01x06, Q1 PSMN8R5-40MSDX, Q2 PSMN8R5-40MSDX, Q3 PSMN8R5-40MSDX, Q4 PSMN8R5-40MSDX, Q5 PSMN8R5-40MSDX, U1 TPS56339DDC

Commit message: added more
Parts:
- J3, J7: footprint Connector_Molex:Molex_Nano-Fit_105310-xx06_2x03_P2.50mm_Vertical -> Connector_Molex:Molex_Nano-Fit_105309-xx06_1x06_P2.50mm_Vertical
- R_G1, R_G2, R_PD1, R_PD2: moved to F.Cu
- moved R10 22.4 mm to (193.8, 83.8), turned to 0 degrees
- moved TP2 22.0 mm to (157.8, 84.7), turned to 180 degrees
- moved R5 19.9 mm to (159.7, 84.7), turned to 90 degrees
- moved R17 19.1 mm to (172.9, 39.6)
- moved JP1 19.0 mm to (170.3, 40.8)
- moved LVPWR4 18.3 mm to (161.3, 84.7), turned to -90 degrees
- moved TP20 17.0 mm to (157.7, 106.5), turned to 90 degrees
- moved R23 15.1 mm to (157.7, 104.5), turned to 180 degrees
- moved LVPWR10 13.6 mm to (157.8, 102.9), turned to 0 degrees
- moved LVPWR16 11.8 mm to (205.9, 84.7), turned to 90 degrees
- moved R20 10.8 mm to (206.0, 104.1), turned to -90 degrees
- moved TP6 10.7 mm to (157.7, 95.8), turned to -90 degrees
- moved R12 10.6 mm to (171.9, 64.2), turned to 0 degrees
- moved R_PD2 10.3 mm to (193.8, 85.6), turned to 180 degrees
- moved LVPWR5 10.2 mm to (161.3, 88.4)
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Routing:
- net /VIN_24V: track 0.00 -> 22.6 mm, vias 0 -> 1
- net /Fans/FAN_A_NEG: track 29.9 -> 17.3 mm, vias 2 -> 0
- net /RPP_EN12: track 14.4 -> 3.30 mm
- net /D_C: track 38.0 -> 27.8 mm, vias 2 -> 0
- net /PWM_FAN_B: track 45.1 -> 35.3 mm, vias 1 -> 0
- net /FAN_A_TACHO: track 37.9 -> 46.4 mm
- net GND: track 8.70 -> 16.4 mm, vias 17 -> 164
- net /LED: track 29.0 -> 35.6 mm
- net /FAN_B_TACHO: track 43.9 -> 37.2 mm, vias 1 -> 2
- net Net-(U1-FB): track 8.23 -> 14.8 mm
- net /LED1: track 17.5 -> 23.6 mm
- net +24V: track 31.9 -> 26.0 mm, vias 8 -> 12
- net /CAN_P: track 129.7 -> 135.1 mm, vias 1 -> 4
- net /PWM_FAN_A: track 41.9 -> 46.9 mm, vias 1 -> 0
- net /RPP_EN24: track 15.8 -> 12.0 mm, vias 2 -> 0
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- added copper zone on F.Cu, net /RPP_EN12
