File: Power.kicad_sch (KiCad schematic)
At the start: 30 parts, among them IC1 LM74502HDDFR, IC2 LM74502HDDFR, Q3 PSMN8R5-40MSDX, Q4 PSMN8R5-40MSDX

Commit message: schematic
Parts:
- renumbered 24V_TP2 to 12V_TP1
Other:
- moved on the sheet: 12V_TP1, 24V_TP1, C10, C11, C12, C13, C14, C15, C20, C21, C4, C5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

Commit message: changes + ioc
Parts:
- removed 12V_TP1: TestPoint, UTSVT_Special:TestPoint_HEX_3mmID, symbol Connector:TestPoint
- removed C11, C12, C14, C15: 0.1u, Capacitor_SMD:C_0603_1608Metric, symbol Device:C
- removed C13, C21: 10u, Capacitor_SMD:C_0805_2012Metric, symbol Device:C
- removed C20: 1u, Capacitor_SMD:C_0603_1608Metric, symbol Device:C
- removed IC2: LM74502HDDFR, UTSVT_Power:SOT65P280X110-8N, symbol UTSVT_ICs:LM74502HDDFR
- removed Q4: PSMN8R5-40MSDX, UTSVT_Power:PSMN8R5-40MSDX, symbol UTSVT_Power:PSMN8R5-40MSDX
- removed R11, R18: 10k, Resistor_SMD:R_0603_1608Metric, symbol Device:R_US
- removed R12: 100k, Resistor_SMD:R_0603_1608Metric, symbol Device:R_US
- removed R14: 9。5k, Resistor_SMD:R_0603_1608Metric, symbol Device:R_US
- removed R28: 200k, Resistor_SMD:R_0603_1608Metric, symbol Device:R_US
- removed Z1, Z2: SMAF4751A-TP, UTSVT_Passives:SODFL5026X125N, symbol UTSVT_Power:SMAF4749A-TP
- removed Z3, Z4: SMAF4744A, UTSVT_Passives:SODFL5026X125N, symbol UTSVT_Power:SMAF4749A-TP
- C10, C9: value 10u -> 0.1u; footprint Capacitor_SMD:C_0805_2012Metric -> Capacitor_SMD:C_0603_1608Metric
- C4: value 220n -> 1u
- C5: value 22n -> 220n
- C6: value 1u -> 22n
- C7: value 220n -> 10u; footprint Capacitor_SMD:C_0603_1608Metric -> Capacitor_SMD:C_0805_2012Metric
- C8: value 22n -> 10u; footprint Capacitor_SMD:C_0603_1608Metric -> Capacitor_SMD:C_0805_2012Metric
- R13: value 9k -> 10k
Connections:
- net +12V is gone; now on net V_OUT: C9.1
- net 12V_BUS is gone; now on net GND: C8.2
- net GND: now also C4.1, C7.2; no longer C6.1, R13.2
- net at IC1.4 (VCAP): now also C5.2; no longer C4.2
- net at IC1.6 (GATE), Q3.4 (G): now also C6.1; no longer C5.1
- net OV: now reaches IC1.7 (OV)
- net OV: no longer R13.1
- net V_OUT: now reaches C8.1
- net V_OUT: now also 24V_TP1.1, C7.1, IC1.8 (SRC), Q3.10 (D_6), Q3.11 (D_7), Q3.5 (D_1), Q3.6 (D_2), Q3.7 (D_3), Q3.8 (D_4), Q3.9 (D_5)
- removed net +24V: 24V_TP1.1, C10.1, IC1.8 (SRC), Q3.10 (D_6), Q3.11 (D_7), Q3.5 (D_1), Q3.6 (D_2), Q3.7 (D_3), Q3.8 (D_4), Q3.9 (D_5)
- net RPP_EN12 renamed VIN
- net VIN: now also C10.1, Q3.1 (S_1), Q3.2 (S_2), Q3.3 (S_3), R13.1; no longer C7.1
- net RPP_EN24 renamed RPP_EN
- net RPP_EN: now also C4.2, C5.1, R13.2; no longer C4.1
- removed net VIN_24V: C5.2, Q3.1 (S_1), Q3.2 (S_2), Q3.3 (S_3)
Other:
- note added: "Power Protection Circuitry"
- note removed: "Power 12V"
- note removed: "Power 24V"

Commit message: small fix
Changed lines of the file:
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@@
+	(wire
+		(pts
+			(xy 132.08 104.14) (xy 128.27 104.14)
+		)
+		(stroke
+			(width 0)
+			(type default)
+		)
+	)
 	(wire
 		(pts
@@
 	(wire
 		(pts
+			(xy 132.08 96.52) (xy 128.27 96.52)
+		)
+		(stroke
+			(width 0)
+			(type default)
+		)
+	)
+	(wire
+		(pts
 			(xy 133.35 62.23) (xy 139.7 62.23)
 		)
@@
 		(pts
 			(xy 158.75 68.58) (xy 158.75 77.47)
-		)
-		(stroke
-			(width 0)
-			(type default)
-		)
-	)
-	(wire
-		(pts
-			(xy 128.27 104.14) (xy 132.08 104.14)
 		)
 		(stroke
@@
 	(hierarchical_label "OV"
 		(shape input)
-		(at 128.27 96.52 0)
+		(at 132.08 96.52 0)
 		(effects
 			(font

Commit message: layout
Parts:
- 24V_TP1: footprint UTSVT_Special:TestPoint_HEX_3mmID -> TestPoint:TestPoint_Pad_1.0x1.0mm
- C10, C9: footprint Capacitor_SMD:C_0603_1608Metric -> Capacitor_SMD:C_0603_1608Metric_Pad1.08x0.95mm_HandSolder; Manufacturer_Part_Number (none) -> MLASH168SB7104KTNA01
- C4: footprint Capacitor_SMD:C_0603_1608Metric -> Capacitor_SMD:C_0603_1608Metric_Pad1.08x0.95mm_HandSolder; Manufacturer_Part_Number (none) -> MLASU168SB5105KTNA01
- C5: footprint Capacitor_SMD:C_0603_1608Metric -> Capacitor_SMD:C_0603_1608Metric_Pad1.08x0.95mm_HandSolder; Manufacturer_Part_Number (none) -> MSASU168SB7224KTNB25
- C6: footprint Capacitor_SMD:C_0603_1608Metric -> Capacitor_SMD:C_0603_1608Metric_Pad1.08x0.95mm_HandSolder; Manufacturer_Part_Number (none) -> 06035C223K4T4A
- C7, C8: footprint Capacitor_SMD:C_0805_2012Metric -> Capacitor_SMD:C_0805_2012Metric_Pad1.18x1.45mm_HandSolder; Manufacturer_Part_Number (none) -> GRM21BR61H106KE43K
- R13: footprint Resistor_SMD:R_0603_1608Metric -> Resistor_SMD:R_0603_1608Metric_Pad0.98x0.95mm_HandSolder; Manufacturer_Part_Number (none) -> CRCW060310K0FKEI
Other:
- moved on the sheet: 24V_TP1, C10, C8, C9

Commit message: fon
Parts:
- removed 24V_TP1: TestPoint, TestPoint:TestPoint_Pad_1.0x1.0mm, symbol Connector:TestPoint
- removed Q3: PSMN8R5-40MSDX, UTSVT_Power:PSMN8R5-40MSDX, symbol UTSVT_Power:PSMN8R5-40MSDX
- added Q6: PSMN8R5-40MSDX, UTSVT_Power:PSMN8R5-40MSDX, symbol utsvt_power:PSMN8R5-40MSDX
- C6: value 22n -> .1u
Connections:
- net GND: now also C6.1
- net VIN: now also Q6.3 (D)
- net V_OUT: now also Q6.1 (S)
- net at IC1.6 (GATE): now also Q6.2 (G); no longer C6.1
Other:
- moved on the sheet: C6

Commit message: Hello
Other:
- moved on the sheet: Q6
Changed lines of the file:
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@@
 	(text "Overvoltage Protection: 29.03V\nVovr = (R2 * Vov)/(R1 + R2)\nVov = Vovr * (R1 + R2) / R2\n29.03 = 1.25 * (200k + 9k) / 9k"
 		(exclude_from_sim no)
-		(at 171.704 99.314 0)
+		(at 171.45 99.06 0)
 		(effects
 			(font
@@
 	(text "Overvoltage Protection: 14.41V\nVovr = (R2 * Vov)/(R1 + R2)\nVov = Vovr * (R1 + R2) / R2\n14.41 = 1.25 * (100k + 9.5k) / 9.5k"
 		(exclude_from_sim no)
-		(at 171.958 110.236 0)
+		(at 171.45 110.49 0)
 		(effects
 			(font
@@
 	(text "R2 : 9.5k\nR1: 100k"
 		(exclude_from_sim no)
-		(at 170.688 117.602 0)
+		(at 170.18 118.11 0)
 		(effects
 			(font
@@
 	(text "24V Input\nBypass Cap"
 		(exclude_from_sim no)
-		(at 161.544 87.376 0)
+		(at 161.29 87.63 0)
 		(effects
 			(font
@@
 	)
 	(junction
-		(at 86.36 57.15)
-		(diameter 0)
-		(color 0 0 0 0)
-	)
-	(junction
 		(at 128.27 62.23)
 		(diameter 0)
@@
 	)
 	(junction
+		(at 86.36 57.785)
+		(diameter 0)
+		(color 0 0 0 0)
+	)
+	(junction
 		(at 81.28 57.15)
 		(diameter 0)
@@
 	(wire
 		(pts
-			(xy 128.27 57.15) (xy 128.27 62.23)
+			(xy 128.27 57.785) (xy 128.27 62.23)
+		)
+		(stroke
+			(width 0)
+			(type default)
+		)
+	)
+	(wire
+		(pts
+			(xy 72.39 57.15) (xy 81.28 57.15)
+		)
+		(stroke
+			(width 0)
+			(type default)
+		)
+	)
+	(wire
+		(pts
+			(xy 104.14 63.5) (xy 104.14 80.01)
 		)
 		(stroke
@@
 	(wire
 		(pts
-			(xy 128.27 57.15) (xy 112.395 57.15)
+			(xy 128.27 57.785) (xy 109.855 57.785)
 		)
 		(stroke
@@
 	(wire
 		(pts
-			(xy 86.36 72.39) (xy 86.36 57.15)
+			(xy 86.36 57.15) (xy 86.36 57.785)
 		)
 		(stroke
@@
 	(wire
 		(pts
-			(xy 76.2 57.15) (xy 81.28 57.15)
-		)
-		(stroke
-			(width 0)
-			(type default)
-		)
-	)
-	(wire
-		(pts
 			(xy 175.26 66.04) (xy 175.26 74.93)
 		)
@@
 		)
 	)
+	(wire
+		(pts
+			(xy 98.425 57.785) (xy 86.36 57.785)
+		)
+		(stroke
+			(width 0)
+			(type default)
+		)
+	)
 	(polyline
 		(pts
@@
 	(wire
 		(pts
-			(xy 106.68 80.01) (xy 109.22 80.01)
-		)
-		(stroke
-			(width 0)
-			(type default)
-		)
-	)
-	(wire
-		(pts
 			(xy 81.28 57.15) (xy 86.36 57.15)
 		)
@@
 	(wire
 		(pts
+			(xy 104.14 80.01) (xy 109.22 80.01)
+		)
+		(stroke
+			(width 0)
+			(type default)
+		)
+	)
+	(wire
+		(pts
 			(xy 139.7 62.23) (xy 143.51 62.23)
 		)
@@
 	(wire
 		(pts
-			(xy 106.68 63.5) (xy 106.68 80.01)
-		)
-		(stroke
-			(width 0)
-			(type default)
-		)
-	)
-	(wire
-		(pts
 			(xy 175.26 50.8) (xy 175.26 58.42)
 		)
@@
 	(wire
 		(pts
-			(xy 100.965 57.15) (xy 100.965 57.785)
-		)
-		(stroke
-			(width 0)
-			(type default)
-		)
-	)
-	(wire
-		(pts
 			(xy 185.42 50.8) (xy 185.42 58.42)
 		)
@@
 	(wire
 		(pts
-			(xy 86.36 57.15) (xy 100.965 57.15)
-		)
-		(stroke
-			(width 0)
-			(type default)
-		)
-	)
-	(wire
-		(pts
 			(xy 162.56 66.04) (xy 162.56 74.93)
 		)
@@
 	(wire
 		(pts
-			(xy 112.395 57.15) (xy 112.395 57.785)
-		)
-		(stroke
-			(width 0)
-			(type default)
-		)
-	)
-	(wire
-		(pts
 			(xy 162.56 50.8) (xy 162.56 58.42)
+		)
+		(stroke
+			(width 0)
+			(type default)
+		)
+	)
+	(wire
+		(pts
+			(xy 86.36 57.785) (xy 86.36 72.39)
 		)
 		(stroke
@@
 	(symbol
 		(lib_id "utsvt_power:PSMN8R5-40MSDX")
-		(at 106.68 57.15 0)
+		(at 104.14 57.15 0)
 		(mirror y)
 		(unit 1)
@@
 		(fields_autoplaced yes)
 		(property "Reference" "Q6"
-			(at 106.68 49.53 0)
+			(at 104.14 49.53 0)
 			(effects
 				(font
@@
 		)
 		(property "Value" "PSMN8R5-40MSDX"
-			(at 106.68 52.07 0)
+			(at 104.14 52.07 0)
 			(effects
 				(font
@@
 		)
 		(property "Footprint" "UTSVT_Power:PSMN8R5-40MSDX"
-			(at 85.09 152.07 0)
+			(at 82.55 152.07 0)
 			(effects
 				(font
@@
 		)
 		(property "Datasheet" "https://assets.nexperia.com/documents/data-sheet/PSMN8R5-40MSD.pdf"
-			(at 85.09 252.07 0)
+			(at 82.55 252.07 0)
 			(effects
 				(font
@@
 		)
 		(property "Description" "MOSFETs PSMN8R5-40MSD/SOT1210/mLFPAK"
-			(at 105.664 45.72 0)
+			(at 103.124 45.72 0)
 			(effects
 				(font
@@
 		)
 		(property "Height" "1"
-			(at 85.09 452.07 0)
+			(at 82.55 452.07 0)
 			(effects
 				(font
@@
 		)
 		(property "Mouser Part Number" "771-PSMN8R5-40MSDX"
-			(at 85.09 552.07 0)
+			(at 82.55 552.07 0)
 			(effects
 				(font
@@
 		)
 		(property "Mouser Price/Stock" "https://www.mouser.co.uk/ProductDetail/Nexperia/PSMN8R5-40MSDX?qs=vHuUswq2%252BswjdnYdBdHaPw%3D%3D"
-			(at 85.09 652.07 0)
+			(at 82.55 652.07 0)
 			(effects
 				(font
@@
 		)
 		(property "Manufacturer_Name" "Nexperia"
-			(at 85.09 752.07 0)
+			(at 82.55 752.07 0)
 			(effects
 				(font
@@
 		)
 		(property "Manufacturer_Part_Number" "PSMN8R5-40MSDX"
-			(at 85.09 852.07 0)
-			(effects
-				(font
+			(at 82.55 852.07 0)
+			(effects
+				(font
