File: StatusLEDs.kicad_sch (KiCad schematic)
At the start: 18 parts

Commit message: layout
Parts:
- R23, R24, R26, R27, R28, R29: value 5k -> 4.3k; footprint (none) -> Resistor_SMD:R_0603_1608Metric_Pad0.98x0.95mm_HandSolder; Manufacturer_Part_Number (none) -> CRCW06034K30FKEA
- TP10, TP16, TP17, TP18, TP19, TP20: footprint (none) -> TestPoint:TestPoint_Pad_1.0x1.0mm
