File: Fuses.kicad_sch (KiCad schematic)
At the start: 5 parts

Commit message: changes + ioc
Parts:
- removed C_R1: 2.26k, Resistor_SMD:R_0805_2012Metric, symbol Device:R_US
- removed C_U1: EL3H7, Package_SO:SOP-4_4.4x2.6mm_P1.27mm, symbol Isolator:SFH617A-1
- added 12V: SMAF4742A, UTSVT_Passives:SODFL5026X125N, symbol UTSVT_Power:SMAF4749A-TP
- added Q2: BUK6M61-60P, symbol Simulation_SPICE:PMOS
- added R_G3: 100, symbol Device:R
- added R_PD3: 10k, symbol Device:R
- C_R2: value 1075k -> 5k
Connections:
- net +24V: now also 12V.1 (K), Q2.3 (S); no longer C_R2.1
- net FANS_POS: now also R_G3.2
- net GND: now also R_PD3.1
- new net: C_R2.1, Q2.1 (D)
- new net: 12V.2 (A), Q2.2 (G), R_G3.1, R_PD3.2
Other:
- note removed: "22.6(.01) = .226W"
- note removed: "C_R1 = (24V - 1.4V)/.01A = 2260Ω"
- note removed: "C_R2 = (24V - 2.5V)/.02A = 1075Ω"
- moved on the sheet: C_D1, C_R2

Commit message: layout
Parts:
- removed Q2: BUK6M61-60P, symbol Simulation_SPICE:PMOS
- added Q2: PSMN8R5-40MSDX, UTSVT_Power:PSMN8R5-40MSDX, symbol UTSVT_Power:PSMN8R5-40MSDX
- C_F1: footprint footprints:3588 -> Fuse:FUSE_3568
- C_R2: value 5k -> 4.3k; Manufacturer_Part_Number (none) -> CRCW06034K30FKEA
- R_G3: footprint (none) -> Resistor_SMD:R_0603_1608Metric_Pad0.98x0.95mm_HandSolder; Manufacturer_Part_Number (none) -> CRCW0603120RFKEC
- R_PD3: footprint (none) -> Resistor_SMD:R_0603_1608Metric_Pad0.98x0.95mm_HandSolder; Manufacturer_Part_Number (none) -> CRCW060310K0FKEI
- renumbered 12V to 12V1
Connections:
- net +24V: now also Q2.1 (S_1), Q2.2 (S_2), Q2.3 (S_3)
- net at C_R2.1: now also Q2.10 (D_6), Q2.11 (D_7), Q2.5 (D_1), Q2.6 (D_2), Q2.7 (D_3), Q2.8 (D_4), Q2.9 (D_5)
- net at 12V1.2 (A), R_G3.1, R_PD3.2: now also Q2.4 (G)
Other:
- note added: "D"
- note added: "G"
- note added: "S"
- moved on the sheet: 12V1, C_D1, C_F1, C_R2, R_G3, R_PD3

Commit message: fon
Parts:
- Q2: footprint UTSVT_Power:PSMN8R5-40MSDX -> UTSVT_Passives:BUK9M34100EX
Connections:
- net FANS_POS renamed FANS_IN
Changed lines of the file:
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@@
 		)
 	)
-	(hierarchical_label "FANS_POS"
+	(hierarchical_label "FANS_IN"
 		(shape input)
 		(at 78.74 59.69 0)
@@
 			)
 		)
-		(property "Footprint" "UTSVT_Power:PSMN8R5-40MSDX"
+		(property "Footprint" "UTSVT_Passives:BUK9M34100EX"
 			(at 134.62 160.96 0)
 			(effects

Commit message: done
Parts:
- Q2: value PSMN8R5-40MSDX -> 771-BUK6M61-60PX; Mouser Part Number 771-PSMN8R5-40MSDX -> 771-BUK6M61-60PX
Changed lines of the file:
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@@
+			)
+		)
+		(property "Sim.Type" ""
+			(at 91.44 83.82 90)
+			(effects
+				(font
+					(size 1.27 1.27)
+				)
+				(hide yes)
 			)
 		)
@@
 		)
 		(property "Mouser Link" ""
+			(at 143.51 96.52 0)
+			(effects
+				(font
+					(size 1.27 1.27)
+				)
+				(hide yes)
+			)
+		)
+		(property "Sim.Type" ""
 			(at 143.51 96.52 0)
 			(effects
@@
 			)
 		)
+		(property "Sim.Type" ""
+			(at 143.51 87.63 0)
+			(effects
+				(font
+					(size 1.27 1.27)
+				)
+				(hide yes)
+			)
+		)
 		(pin "1"
 		)
@@
 			)
 		)
+		(property "Sim.Type" ""
+			(at 67.31 59.69 90)
+			(effects
+				(font
+					(size 1.27 1.27)
+				)
+				(hide yes)
+			)
+		)
 		(pin "1"
 		)
@@
 			)
 		)
-		(property "Value" "PSMN8R5-40MSDX"
+		(property "Value" "771-BUK6M61-60PX"
 			(at 125.73 61.595 0)
 			(effects
@@
 			)
 		)
-		(property "Datasheet" "https://assets.nexperia.com/documents/data-sheet/PSMN8R5-40MSD.pdf"
+		(property "Datasheet" "https://www.mouser.com/ProductDetail/Nexperia/BUK6M61-60PX?qs=olJun0bQHM81LdZ7v5%252BDQQ%3D%3D&srsltid=AfmBOoq3fENficZeHwPsYPzVpNPJVRJ7828S54IrZ1gjzCZoGfPiKI1D"
 			(at 134.62 260.96 0)
 			(effects
@@
 			)
 		)
-		(property "Mouser Part Number" "771-PSMN8R5-40MSDX"
+		(property "Mouser Part Number" "771-BUK6M61-60PX"
 			(at 134.62 560.96 0)
 			(effects
@@
 		)
 		(property "Mouser Link" ""
+			(at 113.03 66.04 0)
+			(effects
+				(font
+					(size 1.27 1.27)
+				)
+				(hide yes)
+			)
+		)
+		(property "Sim.Type" ""
 			(at 113.03 66.04 0)
 			(effects
@@
 			)
 		)
+		(property "Sim.Type" ""
+			(at 83.82 77.47 90)
+			(effects
+				(font
+					(size 1.27 1.27)
+				)
+				(hide yes)
+			)
+		)
 		(pin "2"
 		)
@@
 			(at 91.44 64.77 90)
 			(effects
+				(font
+					(size 1.27 1.27)
+				)
+				(hide yes)
+			)
+		)
+		(property "Sim.Type" ""
+			(at 91.44 64.77 90)
+			(effects

Commit message: fuse mouser part number
Parts:
- C_F1: Mouser Part Number (none) -> 534-3568
Changed lines of the file:
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@@
+			)
+		)
+		(property "Mouser Part Number" "534-3568"
+			(at 67.31 59.69 90)
+			(effects
+				(font
+					(size 1.27 1.27)
+				)
+				(hide yes)
 			)
 		)
