File: PS-MotorControllerInterfacePCB.kicad_sch (KiCad schematic)
At the start: 45 parts, among them J1 53307-2471, J2 MotorController-in, J3 Conn_01x06, J4 PEAK, J5 Power MPPT, J6 MotorController-out

Commit message: fon
Parts:
- added 12V2: TP_12V, TestPoint:TestPoint_Pad_1.0x1.0mm, symbol Connector:TestPoint
- renumbered D_C to D_C1, Fault to Fault1, Message to Message1, OVC to OVC1
Connections:
- net +12V: now also 12V2.1
Other:
- sheet Fuse ports: added FANS_IN; removed FANS_POS
Changed lines of the file:
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@@
 	)
 	(junction
+		(at 209.55 125.73)
+		(diameter 0)
+		(color 0 0 0 0)
+	)
+	(junction
 		(at 264.16 76.2)
 		(diameter 0)
@@
 	(wire
 		(pts
-			(xy 209.55 124.46) (xy 209.55 127)
+			(xy 209.55 124.46) (xy 209.55 125.73)
 		)
 		(stroke
@@
 	(wire
 		(pts
+			(xy 209.55 125.73) (xy 209.55 127)
+		)
+		(stroke
+			(width 0)
+			(type default)
+		)
+	)
+	(wire
+		(pts
 			(xy 199.39 124.46) (xy 199.39 127)
 		)
@@
 	(wire
 		(pts
-			(xy 237.49 21.59) (xy 241.3 21.59)
-		)
-		(stroke
-			(width 0)
-			(type default)
-		)
-	)
-	(wire
-		(pts
 			(xy 90.17 54.61) (xy 101.6 54.61)
 		)
@@
 	(wire
 		(pts
+			(xy 237.49 21.59) (xy 241.3 21.59)
+		)
+		(stroke
+			(width 0)
+			(type default)
+		)
+	)
+	(wire
+		(pts
 			(xy 90.17 62.23) (xy 93.98 62.23)
 		)
@@
 		)
 	)
+	(label "FANS_IN"
+		(at 191.77 21.59 180)
+		(effects
+			(font
+				(size 1.27 1.27)
+			)
+			(justify right bottom)
+		)
+	)
 	(label "PWM_FAN_A"
 		(at 101.6 64.77 0)
@@
 		)
 	)
+	(label "FANS_IN"
+		(at 237.49 21.59 180)
+		(effects
+			(font
+				(size 1.27 1.27)
+			)
+			(justify right bottom)
+		)
+	)
 	(label "LED4"
 		(at 237.49 43.18 180)
@@
 	)
 	(symbol
+		(lib_id "Connector:TestPoint")
+		(at 209.55 125.73 90)
+		(unit 1)
+		(exclude_from_sim no)
+		(in_bom yes)
+		(on_board yes)
+		(dnp no)
+		(property "Reference" "12V2"
+			(at 205.232 121.158 90)
+			(effects
+				(font
+					(size 1.27 1.27)
+				)
+			)
+		)
+		(property "Value" "TP_12V"
+			(at 205.232 123.698 90)
+			(effects
+				(font
+					(size 1.27 1.27)
+				)
+			)
+		)
+		(property "Footprint" "TestPoint:TestPoint_Pad_1.0x1.0mm"
+			(at 209.55 120.65 0)
+			(effects
+				(font
+					(size 1.27 1.27)
+				)
+				(hide yes)
+			)
+		)
+		(property "Datasheet" "~"
+			(at 209.55 120.65 0)
+			(effects
+				(font
+					(size 1.27 1.27)
+				)
+				(hide yes)
+			)
+		)
+		(property "Description" "test point"
+			(at 209.55 125.73 0)
+			(effects
+				(font
+					(size 1.27 1.27)
+				)
+				(hide yes)
+			)
+		)
+		(property "Manufacturer" ""
+			(at 209.55 125.73 90)
+			(effects
+				(font
+					(size 1.27 1.27)
+				)
+				(hide yes)
+			)
+		)
+		(property "Mouser Link" ""
+			(at 209.55 125.73 90)
+			(effects
+				(font
+					(size 1.27 1.27)
+				)
+				(hide yes)
+			)
+		)
+		(pin "1"
+		)
+		(instances
+			(project "PS-MotorControllerInterfacePCB"
+				(path "/a2e13c19-ff3a-4e43-a7f5-200fd5b2b978"
+					(reference "12V2")
+					(unit 1)
+				)
+			)
+		)
+	)
+	(symbol
 		(lib_id "power:+3V3")
 		(at 95.25 27.94 0)
@@
 		(on_board yes)
 		(dnp no)
-		(property "Reference" "OVC"
+		(property "Reference" "OVC1"
 			(at 237.744 121.158 90)
 			(effects
@@
 			(project "PS-MotorControllerInterfacePCB"
 				(path "/a2e13c19-ff3a-4e43-a7f5-200fd5b2b978"
-					(reference "OVC")
+					(reference "OVC1")
 					(unit 1)
 				)
@@
 		(on_board yes)
 		(dnp no)
-		(property "Reference" "D_C"
+		(property "Reference" "D_C1"
 			(at 246.888 120.904 90)
 			(effects
@@
 			(project "PS-MotorControllerInterfacePCB"
 				(path "/a2e13c19-ff3a-4e43-a7f5-200fd5b2b978"
-					(reference "D_C")
+					(reference "D_C1")
 					(unit 1)
 				)
@@
 	)
 	(symbol
-		(lib_id "power:+24V")
-		(at 237.49 21.59 0)
-		(unit 1)
-		(exclude_from_sim no)
-		(in_bom yes)
-		(on_board yes)
-		(dnp no)
-		(property "Reference" "#PWR057"
-			(at 237.49 25.4 0)
-			(effects
-				(font
-					(size 1.27 1.27)
-				)
-				(hide yes)
-			)
-		)
-		(property "Value" "+24V"
-			(at 237.49 17.526 0)
-			(effects
-				(font
-					(size 1.27 1.27)
-				)
-			)
-		)
-		(property "Footprint" ""
-			(at 237.49 21.59 0)
-			(effects
-				(font
-					(size 1.27 1.27)
-				)
-				(hide yes)
-			)
-		)
-		(property "Datasheet" ""
-			(at 237.49 21.59 0)
-			(effects
-				(font
-					(size 1.27 1.27)
-				)
-				(hide yes)
-			)
-		)
-		(property "Description" "Power symbol creates a global label with name \"+24V\""
-			(at 237.49 21.59 0)
-			(effects
-				(font
-					(size 1.27 1.27)
-				)
-				(hide yes)
-			)
-		)
-		(pin "1"
-		)
-		(instances
-			(project "PS-MotorControllerInterfacePCB"
-				(path "/a2e13c19-ff3a-4e43-a7f5-200fd5b2b978"
-					(reference "#PWR057")
-					(unit 1)
-				)
-			)
-		)
-	)
-	(symbol
 		(lib_id "utsvt_connectors:PeripheralSOMConnector")
 		(at 72.39 20.32 0)
@@
 	)
 	(symbol
-		(lib_id "power:+24V")
-		(at 191.77 21.59 0)
-		(unit 1)
-		(exclude_from_sim no)
-		(in_bom yes)
-		(on_board yes)
-		(dnp no)
-		(property "Reference" "#PWR050"
-			(at 191.77 25.4 0)
-			(effects
-				(font
-					(size 1.27 1.27)
-				)
-				(hide yes)
-			)
-		)
-		(property "Value" "+24V"
-			(at 191.516 17.018 0)
-			(effects
-				(font
-					(size 1.27 1.27)
-				)
-			)
-		)
-		(property "Footprint" ""
-			(at 191.77 21.59 0)
-			(effects
-				(font
-					(size 1.27 1.27)
-				)
-				(hide yes)
-			)
-		)
-		(property "Datasheet" ""
-			(at 191.77 21.59 0)
-			(effects
-				(font
-					(size 1.27 1.27)
-				)
-				(hide yes)
-			)
-		)
-		(property "Description" "Power symbol creates a global label with name \"+24V\""
-			(at 191.77 21.59 0)
-			(effects
-				(font
-					(size 1.27 1.27)
-				)
-				(hide yes)
-			)
-		)
-		(pin "1"
-		)
-		(instances
-			(project ""
-				(path "/a2e13c19-ff3a-4e43-a7f5-200fd5b2b978"
-					(reference "#PWR050")
-					(unit 1)
-				)
-			)
-		)
-	)
-	(symbol
 		(lib_id "Connector:TestPoint")
 		(at 261.62 125.73 90)
@@
 		(on_board yes)
 		(dnp no)
-		(property "Reference" "Fault"
+		(property "Reference" "Fault1"
 			(at 257.048 120.904 90)
 			(effects
@@
 			(project "PS-MotorControllerInterfacePCB"
 				(path "/a2e13c19-ff3a-4e43-a7f5-200fd5b2b978"
-					(reference "Fault")
+					(reference "Fault1")
 					(unit 1)
 				)
@@
 		(on_board yes)
 		(dnp no)
-		(property "Reference" "Message"
+		(property "Reference" "Message1"
 			(at 226.822 121.158 90)
 			(effects
@@
 			(project "PS-MotorControllerInterfacePCB"
 				(path "/a2e13c19-ff3a-4e43-a7f5-200fd5b2b978"
-					(reference "Message")
+					(reference "Message1")
 					(unit 1)
 				)
@@
 			)
 		)
-		(pin "FANS_POS" input
+		(pin "FANS_IN" input
 			(at 241.3 21.59 180)
 			(effects

Commit message: done
Parts:
- removed H3: MountingHole_Pad, MountingHole:MountingHole_3.2mm_M3, symbol Mechanical:MountingHole_Pad
- removed TVS1: PTVS5V0Z1USK, Diode_SMD:Nexperia_DSN1608-2_1.6x0.8mm, symbol Diode:PTVS5V0Z1USK
- added Z5: SMAF4749A, UTSVT_Passives:SODFL5026X125N, symbol UTSVT_Power:SMAF4749A-TP
- J3: value Conn_01x06 -> PWR + CAN; Mouser Part Number (none) -> 538-105309-1206
- J4, J5: Mouser Part Number (none) -> 538-105309-1202
- Moco-in1: renamed from J2; Mouser Part Number (none) -> 538-43045-0600
- Moco-out1: renamed from J6; Mouser Part Number (none) -> 538-43045-0600
- Z1, Z2: Mouser Part Number 833-SMAF4749A-TP -> 833-SMAF4751A-TP
- Z3, Z4: Mouser Part Number 833-SMAF4749A-TP -> 833-SMAF4744A-TP
Connections:
- net GND: now also Z5.2 (A)
- net VIN_24V: now also Z5.1 (K)
- no-connect marks 17 -> 16
