File: Hardware/Fuses.kicad_sch (KiCad schematic)
At the start: 7 parts, among them Q2 771-BUK6M61-60PX

Commit message: hi
Parts:
- C_F1: now left out of the parts list
Changed lines of the file:
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@@
 		(unit 1)
 		(exclude_from_sim no)
-		(in_bom yes)
+		(in_bom no)
 		(on_board yes)
 		(dnp no)
