File: Hardware/KiCad/PS-MotorControllerInterfacePCB.kicad_pcb (KiCad board)
At the start: 2 copper layers, 59.1 x 75.7 mm, 126 parts, among them IC1 LM74502HDDFR, IC2 LM74502HDDFR, J1 53307-2471, Q1 PSMN8R5-40MSDX, Q2 BUK6M61-60, Q5 PSMN8R5-40MSDX, Q6 PSMN8R5-40MSDX, Q7 PSMN8R5-40MSDX, U1 TPS56339DDC

Commit message: software pr
Parts:
- moved C11 0.38 mm to (176.7, 66.2)
- moved C14 0.38 mm to (176.6, 75.0)
- moved C15 0.38 mm to (178.6, 75.0)
- moved R14 0.38 mm to (183.2, 68.7)
- moved R18 0.38 mm to (183.2, 71.8)
- moved Z1 0.38 mm to (188.3, 67.7)
- moved C13 0.38 mm to (183.2, 70.2)
- moved C20 0.38 mm to (181.8, 75.1)
- moved C21 0.38 mm to (185.8, 68.2)
- moved IC2 0.38 mm to (179.2, 69.3)
- moved R25 0.38 mm to (177.6, 72.2)
- moved Z2 0.38 mm to (179.2, 63.9)
- moved C12 0.38 mm to (176.7, 69.8)
Changed lines of the file:
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@@
 	(footprint "UTSVT_Power:SOT65P280X110-8N"
 		(layer "F.Cu")
-		(at 179.1 68.95 -90)
+		(at 179.25 69.3 -90)
 		(descr "DDF0008A")
 		(tags "Integrated Circuit")
@@
 	(footprint "Capacitor_SMD:C_0603_1608Metric_Pad1.08x0.95mm_HandSolder"
 		(layer "F.Cu")
-		(at 183.075 69.875)
+		(at 183.225 70.225)
 		(descr "Capacitor SMD 0603 (1608 Metric), square (rectangular) end terminal, IPC-7351 nominal with elongated pad for handsoldering. (Body size source: IPC-SM-782 page 76, https://www.pcb-3d.com/wordpress/wp-content/uploads/ipc-sm-782a_amendment_1_and_2.pdf), generated with kicad-footprint-generator")
 		(tags "capacitor handsolder")
@@
 	(footprint "Capacitor_SMD:C_0603_1608Metric_Pad1.08x0.95mm_HandSolder"
 		(layer "F.Cu")
-		(at 181.6 74.7625 90)
+		(at 181.75 75.1125 90)
 		(descr "Capacitor SMD 0603 (1608 Metric), square (rectangular) end terminal, IPC-7351 nominal with elongated pad for handsoldering. (Body size source: IPC-SM-782 page 76, https://www.pcb-3d.com/wordpress/wp-content/uploads/ipc-sm-782a_amendment_1_and_2.pdf), generated with kicad-footprint-generator")
 		(tags "capacitor handsolder")
@@
 	(footprint "Capacitor_SMD:C_0805_2012Metric_Pad1.18x1.45mm_HandSolder"
 		(layer "F.Cu")
-		(at 176.45 74.6125 90)
+		(at 176.6 74.9625 90)
 		(descr "Capacitor SMD 0805 (2012 Metric), square (rectangular) end terminal, IPC-7351 nominal with elongated pad for handsoldering. (Body size source: IPC-SM-782 page 76, https://www.pcb-3d.com/wordpress/wp-content/uploads/ipc-sm-782a_amendment_1_and_2.pdf, https://docs.google.com/spreadsheets/d/1BsfQQcO9C6DZCsRaXUlFlo91Tg2WpOkGARC1WS5S8t0/edit?usp=sharing), generated with kicad-footprint-generator")
 		(tags "capacitor handsolder")
@@
 	(footprint "Capacitor_SMD:C_0603_1608Metric_Pad1.08x0.95mm_HandSolder"
 		(layer "F.Cu")
-		(at 176.5612 69.4188 90)
+		(at 176.7112 69.7688 90)
 		(descr "Capacitor SMD 0603 (1608 Metric), square (rectangular) end terminal, IPC-7351 nominal with elongated pad for handsoldering. (Body size source: IPC-SM-782 page 76, https://www.pcb-3d.com/wordpress/wp-content/uploads/ipc-sm-782a_amendment_1_and_2.pdf), generated with kicad-footprint-generator")
 		(tags "capacitor handsolder")
@@
 	(footprint "Resistor_SMD:R_0603_1608Metric_Pad0.98x0.95mm_HandSolder"
 		(layer "F.Cu")
-		(at 183.075 71.425 180)
+		(at 183.225 71.775 180)
 		(descr "Resistor SMD 0603 (1608 Metric), square (rectangular) end terminal, IPC-7351 nominal with elongated pad for handsoldering. (Body size source: IPC-SM-782 page 72, https://www.pcb-3d.com/wordpress/wp-content/uploads/ipc-sm-782a_amendment_1_and_2.pdf), generated with kicad-footprint-generator")
 		(tags "resistor handsolder")
@@
 	(footprint "Resistor_SMD:R_0603_1608Metric_Pad0.98x0.95mm_HandSolder"
 		(layer "F.Cu")
-		(at 177.4 71.875 180)
+		(at 177.55 72.225 180)
 		(descr "Resistor SMD 0603 (1608 Metric), square (rectangular) end terminal, IPC-7351 nominal with elongated pad for handsoldering. (Body size source: IPC-SM-782 page 72, https://www.pcb-3d.com/wordpress/wp-content/uploads/ipc-sm-782a_amendment_1_and_2.pdf), generated with kicad-footprint-generator")
 		(tags "resistor handsolder")
@@
 	(footprint "Capacitor_SMD:C_0805_2012Metric_Pad1.18x1.45mm_HandSolder"
 		(layer "F.Cu")
-		(at 178.45 74.6125 90)
+		(at 178.6 74.9625 90)
 		(descr "Capacitor SMD 0805 (2012 Metric), square (rectangular) end terminal, IPC-7351 nominal with elongated pad for handsoldering. (Body size source: IPC-SM-782 page 76, https://www.pcb-3d.com/wordpress/wp-content/uploads/ipc-sm-782a_amendment_1_and_2.pdf, https://docs.google.com/spreadsheets/d/1BsfQQcO9C6DZCsRaXUlFlo91Tg2WpOkGARC1WS5S8t0/edit?usp=sharing), generated with kicad-footprint-generator")
 		(tags "capacitor handsolder")
@@
 	(footprint "UTSVT_Passives:SODFL5026X125N"
 		(layer "F.Cu")
-		(at 179 63.575 90)
+		(at 179.15 63.925 90)
 		(descr "DO-221AC(SMA-FL)")
 		(tags "Zener Diode")
@@
 	(footprint "UTSVT_Passives:SODFL5026X125N"
 		(layer "F.Cu")
-		(at 188.2 67.3 90)
+		(at 188.35 67.65 90)
 		(descr "DO-221AC(SMA-FL)")
 		(tags "Zener Diode")
@@
 	(footprint "Capacitor_SMD:C_0603_1608Metric_Pad1.08x0.95mm_HandSolder"
 		(layer "F.Cu")
-		(at 185.7 67.9 90)
+		(at 185.85 68.25 90)
 		(descr "Capacitor SMD 0603 (1608 Metric), square (rectangular) end terminal, IPC-7351 nominal with elongated pad for handsoldering. (Body size source: IPC-SM-782 page 76, https://www.pcb-3d.com/wordpress/wp-content/uploads/ipc-sm-782a_amendment_1_and_2.pdf), generated with kicad-footprint-generator")
 		(tags "capacitor handsolder")
@@
 	(footprint "Capacitor_SMD:C_0603_1608Metric_Pad1.08x0.95mm_HandSolder"
 		(layer "F.Cu")
-		(at 176.5 65.8 -90)
+		(at 176.65 66.15 -90)
 		(descr "Capacitor SMD 0603 (1608 Metric), square (rectangular) end terminal, IPC-7351 nominal with elongated pad for handsoldering. (Body size source: IPC-SM-782 page 76, https://www.pcb-3d.com/wordpress/wp-content/uploads/ipc-sm-782a_amendment_1_and_2.pdf), generated with kicad-footprint-generator")
 		(tags "capacitor handsolder")
@@
 	(footprint "Resistor_SMD:R_0603_1608Metric_Pad0.98x0.95mm_HandSolder"
 		(layer "F.Cu")
-		(at 183.1 68.3 180)
+		(at 183.25 68.65 180)
 		(descr "Resistor SMD 0603 (1608 Metric), square (rectangular) end terminal, IPC-7351 nominal with elongated pad for handsoldering. (Body size source: IPC-SM-782 page 72, https://www.pcb-3d.com/wordpress/wp-content/uploads/ipc-sm-782a_amendment_1_and_2.pdf), generated with kicad-footprint-generator")
 		(tags "resistor handsolder")
@@
 	)
 	(segment
-		(start 177.4175 67.7)
-		(end 176.5612 68.5563)
+		(start 177.5675 68.05)
+		(end 176.7112 68.9063)
 		(width 0.3)
 		(layer "F.Cu")
@@
 	)
 	(segment
-		(start 178.125 67.7)
-		(end 177.4175 67.7)
+		(start 178.275 68.05)
+		(end 177.5675 68.05)
 		(width 0.3)
 		(layer "F.Cu")

Commit message: revB, will make aesthetic changes
Parts:
- removed 12V: TP_12V, TestPoint:TestPoint_Pad_1.0x1.0mm
- removed 24V: TP_B_NEG, TestPoint:TestPoint_Pad_1.0x1.0mm
- removed 24V, FAN_A_NEG, FAN_B_NEG, LVPWR10, LVPWR11, LVPWR12, LVPWR13, LVPWR14, LVPWR15: LED, LED_SMD:LED_0603_1608Metric
- removed 3V3: TP_3V3, TestPoint:TestPoint_Pad_1.0x1.0mm
- removed C_D1: 20mA, LED_SMD:LED_0805_2012Metric
- removed C_F1: 10A, Fuse:FUSE_3568
- removed C_R2: 4.3k, Resistor_SMD:R_0805_2012Metric
- removed D5, D7: 1N4148WT, Diode_SMD:D_SOD-523
- removed Drive_C: TP_D_C, TestPoint:TestPoint_Pad_1.0x1.0mm
- removed FANS: Conn_01x06, Connector_Molex:Molex_Nano-Fit_105309-xx06_1x06_P2.50mm_Vertical
- removed G***: LOGO, Fuse:richarddd
- removed G***: LHRs_LOGO, UTSVT_Logos:LHRs_LOGO
- removed G***: LOGO, UTSVT_Logos:Hallock_Image
- removed GND: TP_GND, TestPoint:TestPoint_Pad_1.0x1.0mm
- removed H4: MountingHole_Pad, MountingHole:MountingHole_3.2mm_M3
- removed LED: LED, TestPoint:TestPoint_Pad_1.0x1.0mm
- removed Moco-In: MotorController-in, UTSVT_Connectors:Molex_Microfit3.0_02x03_6-Pin-Vertical-PCB-Receptacle_447690601
- removed Moco-out: MotorController-out, UTSVT_Connectors:Molex_Microfit3.0_02x03_6-Pin-Vertical-PCB-Receptacle_447690601
- removed PEAK: PEAK, Connector_Molex:Molex_Nano-Fit_105309-xx02_1x02_P2.50mm_Vertical
- removed PWM_A2: TP_PWM_A, TestPoint:TestPoint_Pad_1.0x1.0mm
- removed PWM_B2: TP_PWM_B, TestPoint:TestPoint_Pad_1.0x1.0mm
- removed PWR + CAN: Conn_01x06, Connector_Molex:Molex_Nano-Fit_105309-xx06_1x06_P2.50mm_Vertical
- removed PWR MPPT: Power MPPT, UTSVT_Connectors:Molex_Nano-Fit_105309-xx02_1x02_P2.50mm_Vertical
- removed R27, R28, R29: 4.3k, Resistor_SMD:R_0603_1608Metric_Pad0.98x0.95mm_HandSolder
- removed R_A_TACH_PD1, R_B_TACH_PD1: 10k, Resistor_SMD:R_0603_1608Metric_Pad0.98x0.95mm_HandSolder
- removed TACH_A: TP_A_TACH, TestPoint:TestPoint_Pad_1.0x1.0mm
- removed TACH_B: TP_B_TACH, TestPoint:TestPoint_Pad_1.0x1.0mm
- removed Term Jumper: TRM, Connector_PinHeader_2.54mm:PinHeader_1x02_P2.54mm_Vertical
- removed Z5: SMAF4744A, UTSVT_Passives:SODFL5026X125N
- added 24V1: TP_24V, TestPoint:TestPoint_Pad_1.0x1.0mm, F.Cu at (154.6, 45.6)
- added 3V1: TP_3V3, TestPoint:TestPoint_Pad_1.0x1.0mm, F.Cu at (155.5, 93.6)
- added C19: .1u, Capacitor_SMD:C_0603_1608Metric_Pad1.08x0.95mm_HandSolder, F.Cu at (190.0, 45.6)
- added C22: 10u, Capacitor_SMD:C_0805_2012Metric_Pad1.18x1.45mm_HandSolder, F.Cu at (176.8, 44.5)
- added C23: 0.1u, Capacitor_SMD:C_0603_1608Metric_Pad1.08x0.95mm_HandSolder, F.Cu at (181.9, 48.9)
- added D1: 1N4148WT, easyeda2kicad:SOD-523F_L1.2-W0.8-LS1.7-RD, F.Cu at (174.0, 98.3)
- added D2: 1N4148WT, easyeda2kicad:SOD-523F_L1.2-W0.8-LS1.7-RD, F.Cu at (179.0, 98.3)
- added D_C1: TP_D_C, TestPoint:TestPoint_Pad_1.0x1.0mm, F.Cu at (154.4, 61.8)
- added F1: 10A, Moco:FUSE_3568, F.Cu at (198.8, 83.0)
- added H3: MountingHole_Pad, MountingHole:MountingHole_3.2mm_M3, F.Cu at (182.4, 40.2)
- added J2: PWR board, Connector_Molex:Molex_Nano-Fit_105313-xx02_1x02_P2.50mm_Horizontal, F.Cu at (199.8, 38.9)
- added J3: CAN board in, Connector_Molex:Molex_Nano-Fit_105314-xx06_2x03_P2.50mm_Horizontal, F.Cu at (210.0, 97.9)
- added J4: 53307-2471, UTSVT_Connectors:PeripheralSOM, F.Cu at (175.4, 85.9)
- added J5: PWR Moco, Connector_Molex:Molex_Nano-Fit_105313-xx02_1x02_P2.50mm_Horizontal, F.Cu at (207.5, 64.6)
- added J6: Candapter, Connector_Molex:Molex_Nano-Fit_105313-xx02_1x02_P2.50mm_Horizontal, F.Cu at (196.7, 100.4)
- added J7: CAN board -> mppt +moco, Connector_Molex:Molex_Nano-Fit_105313-xx03_1x03_P2.50mm_Horizontal, F.Cu at (209.2, 51.6)
- added J8: CAN mppts + moco -> board, Connector_Molex:Molex_Nano-Fit_105313-xx03_1x03_P2.50mm_Horizontal, F.Cu at (209.5, 38.8)
- added J9: Conn_01x06, Connector_Molex:Molex_Nano-Fit_105313-xx06_1x06_P2.50mm_Horizontal, F.Cu at (181.9, 100.5)
- added JP1: TRM, Connector_PinHeader_2.54mm:PinHeader_1x02_P2.54mm_Vertical, F.Cu at (188.6, 103.1)
- added LED6: LED, LED_SMD:LED_0603_1608Metric, F.Cu at (198.9, 92.9)
- added LED7: LED, LED_SMD:LED_0603_1608Metric, F.Cu at (190.5, 92.8)
- added LVPWR1: LED, LED_SMD:LED_0603_1608Metric, F.Cu at (156.6, 44.4)
- added PD_TACHA1: 10k, Resistor_SMD:R_0603_1608Metric_Pad0.98x0.95mm_HandSolder, F.Cu at (164.9, 105.3)
- added PD_TACHB1: 10k, Resistor_SMD:R_0603_1608Metric_Pad0.98x0.95mm_HandSolder, F.Cu at (164.9, 103.7)
- added PWM_A1: TP_PWM_B, TestPoint:TestPoint_Pad_1.0x1.0mm, F.Cu at (207.6, 87.2)
- added PWM_B1: TP_PWM_A, TestPoint:TestPoint_Pad_1.0x1.0mm, F.Cu at (155.5, 88.1)
- added Q3: NVMFWS1D7N04XMT1G, Package_TO_SOT_SMD:SOT-23, F.Cu at (173.6, 68.4)
- added Q4: NVMFWS1D7N04XMT1G, Package_TO_SOT_SMD:SOT-23, F.Cu at (177.6, 68.8)
- added TACH_A1: TP_PWM_B, TestPoint:TestPoint_Pad_1.0x1.0mm, F.Cu at (188.6, 109.4)
- added TACH_B1: TP_PWM_B, TestPoint:TestPoint_Pad_1.0x1.0mm, F.Cu at (164.8, 109.2)
- added TP1: TP_GND, TestPoint:TestPoint_Pad_1.0x1.0mm, F.Cu at (207.6, 92.8)
- added TP2: LED, TestPoint:TestPoint_Pad_1.0x1.0mm, F.Cu at (154.4, 51.0)
- added TP3: LED1, TestPoint:TestPoint_Pad_1.0x1.0mm, F.Cu at (165.2, 96.3)
- added TP4: LED2, TestPoint:TestPoint_Pad_1.0x1.0mm, F.Cu at (173.6, 96.3)
- added TP5: LED3, TestPoint:TestPoint_Pad_1.0x1.0mm, F.Cu at (182.1, 96.3)
- added TP6: LED4, TestPoint:TestPoint_Pad_1.0x1.0mm, F.Cu at (198.9, 96.5)
- added TP7: LED5, TestPoint:TestPoint_Pad_1.0x1.0mm, F.Cu at (190.5, 96.3)
- 12V1: value SMAF4742A -> TP_12V; footprint UTSVT_Passives:SODFL5026X125N -> TestPoint:TestPoint_Pad_1.0x1.0mm
- C1: value 10u -> .1u; footprint Capacitor_SMD:C_0805_2012Metric_Pad1.18x1.45mm_HandSolder -> Capacitor_SMD:C_0603_1608Metric_Pad1.08x0.95mm_HandSolder
- C10: value 0.1u -> 1u
- C11: value 1u -> 100n
- C12: value 220n -> C_Small
- C13, C6: value .1u -> 10u; footprint Capacitor_SMD:C_0603_1608Metric_Pad1.08x0.95mm_HandSolder -> Capacitor_SMD:C_0805_2012Metric_Pad1.18x1.45mm_HandSolder
- C16: value 100n -> 10u; footprint Capacitor_SMD:C_0603_1608Metric_Pad1.08x0.95mm_HandSolder -> Capacitor_SMD:C_0805_2012Metric_Pad1.18x1.45mm_HandSolder
- C17, C3: value 22u -> .1u; footprint Capacitor_SMD:C_0805_2012Metric_Pad1.18x1.45mm_HandSolder -> Capacitor_SMD:C_0603_1608Metric_Pad1.08x0.95mm_HandSolder
- C18: value 22u -> 1u; footprint Capacitor_SMD:C_0805_2012Metric_Pad1.18x1.45mm_HandSolder -> Capacitor_SMD:C_0603_1608Metric_Pad1.08x0.95mm_HandSolder
- C2: value 100n -> 1u
- C20, C9: value 0.1u -> 220n
- C21: value 0.1u -> 10u; footprint Capacitor_SMD:C_0603_1608Metric_Pad1.08x0.95mm_HandSolder -> Capacitor_SMD:C_0805_2012Metric_Pad1.18x1.45mm_HandSolder
- C4: value 1u -> 220n
- C5: value 220n -> 10u; footprint Capacitor_SMD:C_0603_1608Metric_Pad1.08x0.95mm_HandSolder -> Capacitor_SMD:C_0805_2012Metric_Pad1.18x1.45mm_HandSolder
- C7: value 10u -> 0.1u; footprint Capacitor_SMD:C_0805_2012Metric_Pad1.18x1.45mm_HandSolder -> Capacitor_SMD:C_0603_1608Metric_Pad1.08x0.95mm_HandSolder
- J1: value 53307-2471 -> CAN board out; footprint UTSVT_Connectors:PeripheralSOM -> Connector_Molex:Molex_Nano-Fit_105314-xx06_2x03_P2.50mm_Horizontal
- L1: value 6.8u -> 4.7u; footprint Inductor_SMD:L_6.3x6.3_H3 -> easyeda2kicad:IND-SMD_L5.0-W5.0
- LED1: value LED1 -> 20mA; footprint TestPoint:TestPoint_Pad_1.0x1.0mm -> LED_SMD:LED_0805_2012Metric
- LED2: value LED2 -> LED; footprint TestPoint:TestPoint_Pad_1.0x1.0mm -> LED_SMD:LED_0603_1608Metric
- LED3: value LED3 -> LED; footprint TestPoint:TestPoint_Pad_1.0x1.0mm -> LED_SMD:LED_0603_1608Metric
- LED4: value LED4 -> LED; footprint TestPoint:TestPoint_Pad_1.0x1.0mm -> LED_SMD:LED_0603_1608Metric
- LED5: value LED5 -> LED; footprint TestPoint:TestPoint_Pad_1.0x1.0mm -> LED_SMD:LED_0603_1608Metric
- Q1: value PSMN8R5-40MSDX -> IRLML0030; footprint UTSVT_Power:PSMN8R5-40MSDX -> Package_TO_SOT_SMD:SOT-23
- Q2: value BUK6M61-60 -> IRLML0030; footprint UTSVT_Passives:BUK9M34100EX -> Package_TO_SOT_SMD:SOT-23
- Q5: value PSMN8R5-40MSDX -> 771-BUK6M61-60PX; footprint UTSVT_Power:PSMN8R5-40MSDX -> Moco:BUK9M34100EX
- Q6, Q7: value PSMN8R5-40MSDX -> NVMFWS1D7N04XMT1G; footprint UTSVT_Power:PSMN8R5-40MSDX -> Package_TO_SOT_SMD:SOT-23
- R1: value 30 -> 120
- R10: value 0 -> 100k
- R11: value 100k -> 4.3k
- R12: value 9。5k -> 4.3k; moved to F.Cu
- R13, R14, R9: value 10k -> 4.3k
- R15: value 4.3k -> 0
- R16: value 220k -> 10k; footprint Resistor_SMD:R_0603_1608Metric_Pad0.98x0.95mm_HandSolder -> Resistor_SMD:R_0805_2012Metric_Pad1.20x1.40mm_HandSolder
- R17: value 120 -> 4.3k; footprint Resistor_SMD:R_0603_1608Metric_Pad0.98x0.95mm_HandSolder -> Resistor_SMD:R_0805_2012Metric_Pad1.20x1.40mm_HandSolder
- R18: value 200k -> 100k
- R19: value 4.3k -> 9.09k; moved to F.Cu
- R2: value 140k -> 4.3k
- R20: value 4.3k -> 10k; footprint Resistor_SMD:R_0603_1608Metric_Pad0.98x0.95mm_HandSolder -> Resistor_SMD:R_0805_2012Metric_Pad1.20x1.40mm_HandSolder; moved to F.Cu
- R25: value 9k -> 4.3k
- R4: value 4.3k -> 200k
- R6: value 4.3k -> 9k
- R7: moved to F.Cu
- R8: value 4.3k -> 9。5k
- U1: value TPS56339DDC -> LMR33630ADDA; footprint Package_TO_SOT_SMD:SOT-23-6 -> Package_SO:Texas_HSOP-8-1EP_3.9x4.9mm_P1.27mm_ThermalVias
- Z2: value SMAF4751A-TP -> SMAF4758A
- Z3: value SMAF4744A -> SMAF4758A
- Z4: value SMAF4744A -> SMAF4742A
- moved R7 59.8 mm to (158.0, 67.0), turned to 90 degrees
- moved R4 59.8 mm to (189.4, 51.5), turned to 90 degrees
- moved LED2 57.1 mm to (156.3, 51.0)
- moved R20 54.0 mm to (192.9, 51.8)
- moved LVPWR2 48.4 mm to (199.1, 61.8)
- moved R3 47.2 mm to (197.3, 63.7), turned to -90 degrees
- moved R21 44.7 mm to (158.2, 51.0), turned to 90 degrees
- moved LVPWR6 44.4 mm to (156.3, 61.8), turned to -90 degrees
- moved R19 44.4 mm to (173.2, 52.2), turned to 90 degrees
- moved Fault1 43.2 mm to (154.4, 56.4)
- moved R17 36.1 mm to (186.5, 74.1)
- moved LED1 35.6 mm to (186.5, 77.7), turned to 90 degrees
- moved R1 33.2 mm to (188.6, 100.4), turned to 0 degrees
- moved Z4 33.2 mm to (191.8, 77.2), turned to -90 degrees
- moved R25 30.9 mm to (198.9, 94.6)
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Connections:
- 12V1 pad 1: +24V -> +12V
- C1 pad 1: +24V -> GND
- C1 pad 2: GND -> /12V_BUS
- C10 pad 1: /12V_BUS -> Net-(U1-VCC)
- C11 pad 1: GND -> Net-(U1-BOOT)
- C11 pad 2: /RPP_EN24 -> Net-(U1-SW)
- C12 pad 1: /RPP_EN24 -> /12V_BUS
- C12 pad 2: Net-(IC2-VCAP) -> Net-(U1-FB)
- C13 pad 1: GND -> /12V_BUS
- C13 pad 2: /VIN_24V -> GND
- C14 pad 1: +24V -> /12V_BUS
- C15 pad 1: +24V -> /12V_BUS
- C16 pad 1: Net-(C16-Pad1) -> /12V_BUS
- C16 pad 2: /Buck Converter 24V-12V/SW -> GND
- C17 pad 1: /12V_BUS -> GND
- C17 pad 2: GND -> /VIN_24V
- C18 pad 1: /12V_BUS -> GND
- C18 pad 2: GND -> /RPP_EN24
- C2 pad 1: +24V -> GND
- C2 pad 2: GND -> /RPP_EN12
- C20 pad 1: +24V -> /RPP_EN24
- C20 pad 2: GND -> Net-(IC2-VCAP)
- C21 pad 1: /VIN_24V -> +24V
- C3 pad 1: /12V_BUS -> GND
- C3 pad 2: GND -> /12V_BUS
- C4 pad 1: GND -> /RPP_EN12
- C4 pad 2: /RPP_EN12 -> Net-(IC1-VCAP)
- C5 pad 1: /RPP_EN12 -> +12V
- C5 pad 2: Net-(IC1-VCAP) -> GND
- C6 pad 1: GND -> +12V
- C6 pad 2: /12V_BUS -> GND
- C8 pad 1: +12V -> +24V
- C9 pad 1: +12V -> +24V
- IC1 pad 8: +12V -> Net-(IC1-SRC)
- IC2 pad 8: +24V -> Net-(IC2-SRC)
- J1 pad 1: GND -> /CAN_H
- J1 pad 2: +3V3 -> /CAN_L
- J1 pad 4: /S_OC -> unconnected-(J1-Pin_4-Pad4)
- J1 pad 5: GND -> unconnected-(J1-Pin_5-Pad5)
- J1 pad 6: /MESSAGE -> unconnected-(J1-Pin_6-Pad6)
- L1 pad 1: /Buck Converter 24V-12V/SW -> Net-(U1-SW)
- LED1 pad 1: /LED1 -> GND
- LED2 pad 1: /LED2 -> GND
- LED3 pad 1: /LED3 -> GND
- LED4 pad 1: /LED4 -> GND
- LED5 pad 1: /LED5 -> GND
- Q1 pad 1: GND -> Net-(Q1-G)
- Q1 pad 3: GND -> /Fans/FAN_A_NEG
- Q2 pad 1: +24V -> Net-(Q2-G)
- Q2 pad 2: +24V -> GND
- Q2 pad 3: +24V -> /Fans/FAN_B_NEG
- Q5 pad 1: GND -> +24V
- Q5 pad 10: /Fans/FAN_B_NEG -> Net-(Q5-D_1)
- Q5 pad 11: /Fans/FAN_B_NEG -> Net-(Q5-D_1)
- Q5 pad 2: GND -> +24V
- Q5 pad 3: GND -> +24V
- Q5 pad 5: /Fans/FAN_B_NEG -> Net-(Q5-D_1)
- Q5 pad 6: /Fans/FAN_B_NEG -> Net-(Q5-D_1)
- Q5 pad 7: /Fans/FAN_B_NEG -> Net-(Q5-D_1)
- Q5 pad 8: /Fans/FAN_B_NEG -> Net-(Q5-D_1)
- Q5 pad 9: /Fans/FAN_B_NEG -> Net-(Q5-D_1)
- Q6 pad 1: +12V -> Net-(IC2-GATE)
- Q6 pad 2: Net-(IC1-GATE) -> Net-(IC2-SRC)
- Q6 pad 3: /12V_BUS -> /VIN_24V
- Q7 pad 1: +24V -> Net-(IC2-GATE)
- Q7 pad 2: Net-(IC2-GATE) -> +24V
- Q7 pad 3: /VIN_24V -> Net-(IC2-SRC)
- R1 pad 1: Net-(U1-BOOT) -> /CAN_H
- R1 pad 2: Net-(C16-Pad1) -> Net-(JP1-A)
- R10 pad 1: /PWM_FAN_A -> /Power12V/OV
- R10 pad 2: /PWM_FAN_B -> /12V_BUS
- R11 pad 1: /12V_BUS -> Net-(LVPWR6-A)
- R11 pad 2: /Power12V/OV -> /D_C
- R12 pad 1: /Power12V/OV -> Net-(LVPWR7-A)
- R12 pad 2: GND -> /M_FAULT
- R13 pad 1: /12V_BUS -> Net-(LVPWR8-A)
- R13 pad 2: /RPP_EN12 -> /PWM_FAN_B
- R14 pad 1: /VIN_24V -> Net-(LVPWR9-A)
- R14 pad 2: /RPP_EN24 -> /PWM_FAN_A
- R15 pad 1: Net-(LVPWR6-A) -> /PWM_FAN_A
- R16 pad 1: +24V -> /12V_BUS
- R16 pad 2: Net-(U1-EN) -> /RPP_EN12
- R17 pad 1: /CAN_P -> Net-(Q5-D_1)
- R17 pad 2: Net-(JP1-A) -> Net-(LED1-A)
- R18 pad 1: /VIN_24V -> /12V_BUS
- R18 pad 2: /Power24V/OV -> Net-(U1-FB)
- R19 pad 1: Net-(LVPWR16-A) -> Net-(U1-FB)
- R19 pad 2: +24V -> GND
- R2 pad 1: /12V_BUS -> Net-(LVPWR1-A)
- R2 pad 2: Net-(U1-FB) -> +24V
- R20 pad 1: Net-(LVPWR17-A) -> /VIN_24V
- R20 pad 2: +24V -> /RPP_EN24
- R21 pad 1: Net-(LVPWR8-A) -> Net-(LED2-A)
- R21 pad 2: /D_C -> /LED
- R22 pad 1: Net-(LVPWR9-A) -> Net-(LED3-A)
- R22 pad 2: /M_FAULT -> /LED1
- R23 pad 1: Net-(LVPWR10-A) -> Net-(LED4-A)
- R23 pad 2: /LED -> /LED2
- R24 pad 1: Net-(LVPWR11-A) -> Net-(LED5-A)
- R24 pad 2: /LED1 -> /LED3
- R25 pad 1: /Power24V/OV -> Net-(LED6-A)
- R25 pad 2: GND -> /LED4
- R26 pad 2: /LED2 -> /LED5
- R3 pad 2: +3V3 -> +12V
- R4 pad 1: Net-(LVPWR3-A) -> /Power24V/OV
- R4 pad 2: /PWM_FAN_A -> /VIN_24V
- R5 pad 1: Net-(LVPWR4-A) -> Net-(LVPWR3-A)
- R5 pad 2: /MESSAGE -> +3V3
- R6 pad 1: Net-(LVPWR7-A) -> GND
- R6 pad 2: +12V -> /Power24V/OV
- R7 pad 1: Net-(LVPWR1-A) -> Net-(LVPWR4-A)
- R7 pad 2: +24V -> /MESSAGE
- R8 pad 1: Net-(LVPWR5-A) -> /Power12V/OV
- R8 pad 2: /S_OC -> GND
- R9 pad 1: Net-(U1-FB) -> Net-(LVPWR5-A)
- R9 pad 2: GND -> /S_OC
- R_G1 pad 2: /PWM_FAN_A -> /PWM_FAN_B
- R_G2 pad 1: Net-(Q5-G) -> Net-(Q2-G)
- R_G2 pad 2: /PWM_FAN_B -> /PWM_FAN_A
- R_G3 pad 1: Net-(12V1-A) -> Net-(Q5-G)
- R_PD2 pad 2: Net-(Q5-G) -> Net-(Q2-G)
- R_PD3 pad 2: Net-(12V1-A) -> /FANS_IN
- U1 pad 2: /Buck Converter 24V-12V/SW -> +24V
- U1 pad 4: Net-(U1-FB) -> unconnected-(U1-PG-Pad4)
- U1 pad 5: Net-(U1-EN) -> Net-(U1-FB)
- U1 pad 6: Net-(U1-BOOT) -> Net-(U1-VCC)
- Z4 pad 1: /12V_BUS -> +24V
- Z4 pad 2: GND -> /FANS_IN
Routing:
- net /CAN_L: track 0.00 -> 139.8 mm, vias 0 -> 1
- net /CAN_N: track 133.6 -> 0.00 mm, vias 1 -> 0
- net /CAN_P: track 133.1 -> 0.00 mm, vias 4 -> 0
- net /CAN_H: track 0.00 -> 130.7 mm, vias 0 -> 2
- net /LED4: track 11.6 -> 25.9 mm
- net +3V3: track 50.4 -> 37.2 mm, vias 1 -> 2
- net Net-(12V1-A): track 12.9 -> 0.00 mm, vias 2 -> 0
- net /PWM_FAN_B: track 37.3 -> 25.7 mm
- net /LED2: track 20.8 -> 9.54 mm
- net /LED: track 36.3 -> 46.1 mm
- net Net-(U1-FB): track 15.3 -> 5.61 mm, vias 2 -> 0
- net /M_FAULT: track 30.2 -> 39.8 mm
- net GND: track 17.2 -> 8.06 mm, vias 185 -> 10
- net /FAN_B_TACHO: track 37.0 -> 28.8 mm
- net Net-(U1-SW): track 0.00 -> 8.25 mm
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- added copper zone on F.Cu, net Net-(U1-FB)
- removed copper zone on F.Cu, net /Buck Converter 24V-12V/SW
- removed copper zone on F.Cu, net /Fans/FAN_A_NEG
- removed copper zone on F.Cu, net /Fans/FAN_B_NEG

Commit message: revB layout
Parts:
- removed LVPWR8, LVPWR9: LED, LED_SMD:LED_0603_1608Metric
- removed R13, R14: 4.3k, Resistor_SMD:R_0603_1608Metric_Pad0.98x0.95mm_HandSolder
- moved PWM_B1 52.0 mm to (207.5, 88.4)
- moved R_PD1 24.1 mm to (189.3, 92.4), turned to 0 degrees
- moved Q1 22.1 mm to (189.3, 95.1)
- moved R_PD2 20.5 mm to (165.8, 92.1), turned to 0 degrees
- moved Q2 18.3 mm to (165.8, 94.9)
- moved R_G1 17.8 mm to (189.3, 90.8), turned to 180 degrees
- moved R_G2 13.9 mm to (165.8, 90.6)
- moved R25 13.8 mm to (185.4, 91.7), turned to 0 degrees
- moved TP6 13.6 mm to (185.4, 95.1), turned to 0 degrees
- moved LED6 13.5 mm to (185.4, 93.2)
- moved R26 9.29 mm to (181.6, 91.7), turned to 0 degrees
- moved TP7 8.98 mm to (181.6, 95.0)
- moved LED7 8.88 mm to (181.6, 93.2), turned to 180 degrees
- moved R1 6.55 mm to (188.3, 106.9), turned to 180 degrees
- moved D2 6.42 mm to (172.6, 98.2), turned to 0 degrees
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Connections:
- D1 pad 2: /Fans/FAN_A_NEG -> /Fans/FAN_B_NEG
- D2 pad 2: /Fans/FAN_B_NEG -> /Fans/FAN_A_NEG
- Q1 pad 3: /Fans/FAN_A_NEG -> /Fans/FAN_B_NEG
- Q2 pad 3: /Fans/FAN_B_NEG -> /Fans/FAN_A_NEG
Routing:
- net /CAN_H: track 130.7 -> 154.5 mm, vias 2 -> 0
- net GND: track 8.06 -> 28.6 mm, vias 10 -> 8
- net /PWM_FAN_A: track 39.7 -> 55.2 mm
- net /LED4: track 25.9 -> 13.9 mm
- net /PWM_FAN_B: track 25.7 -> 36.9 mm
- net /LED5: track 18.4 -> 11.3 mm
- net /FAN_A_TACHO: track 51.4 -> 45.3 mm
- net /Fans/FAN_A_NEG: track 17.2 -> 11.6 mm, vias 1 -> 0
- net /CAN_L: track 139.8 -> 145.2 mm, vias 1 -> 0
- net /FAN_B_TACHO: track 28.8 -> 34.1 mm, vias 2 -> 1
- net /LED1: track 16.1 -> 11.8 mm
- net /FANS_IN: track 56.3 -> 59.8 mm
- net /LED3: track 10.9 -> 7.47 mm
- net +24V: track 16.8 -> 19.8 mm
- net Net-(Q2-G): track 6.32 -> 3.39 mm
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