File: Hardware/KiCad/PS-MotorControllerInterfacePCB.kicad_pcb (KiCad board)
At the start: 2 copper layers, 59.1 x 75.7 mm, 112 parts, among them IC1 LM74502HDDFR, J1 PWR board, J2 CAN board out, J3 CAN board in, J4 Candapter, J5 53307-2471, J6 CAN board -> mppt +moco, J7 CAN mppts + moco -> board, J8 PWR Moco, J9 Conn_01x06, Q1 IRLML0030, Q2 IRLML0030, Q3 NVMFWS1D7N04XMT1G, Q4 NVMFWS1D7N04XMT1G, U1 LMR33630ADDA, U2 TPS27SA08-Q1

Commit message: changes
Routing:
- net GND: vias 223 -> 200
Changed lines of the file:
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@@
-	)
-	(via
-		(at 162.928572 44.9)
-		(size 0.6)
-		(drill 0.3)
-		(layers "F.Cu" "B.Cu")
-		(free yes)
-		(net 3)
 	)
 	(via
@@
 	)
 	(via
-		(at 173.9 43.6)
-		(size 0.6)
-		(drill 0.3)
-		(layers "F.Cu" "B.Cu")
-		(free yes)
-		(net 3)
-	)
-	(via
 		(at 159.028571 37.5)
 		(size 0.6)
@@
 	)
 	(via
-		(at 179.557143 43.6)
-		(size 0.6)
-		(drill 0.3)
-		(layers "F.Cu" "B.Cu")
-		(free yes)
-		(net 3)
-	)
-	(via
 		(at 192.5 60.5)
 		(size 0.6)
@@
 	)
 	(via
-		(at 185.214286 43.6)
-		(size 0.6)
-		(drill 0.3)
-		(layers "F.Cu" "B.Cu")
-		(free yes)
-		(net 3)
-	)
-	(via
 		(at 167.357143 71.7)
 		(size 0.6)
@@
 	)
 	(via
-		(at 165.757143 46.4)
-		(size 0.6)
-		(drill 0.3)
-		(layers "F.Cu" "B.Cu")
-		(free yes)
-		(net 3)
-	)
-	(via
 		(at 176.957143 68.7)
 		(size 0.6)
@@
 	)
 	(via
-		(at 176.728571 43.6)
-		(size 0.6)
-		(drill 0.3)
-		(layers "F.Cu" "B.Cu")
-		(free yes)
-		(net 3)
-	)
-	(via
 		(at 182.628572 109.4)
 		(size 0.6)
@@
 	)
 	(via
-		(at 182.385714 43.6)
-		(size 0.6)
-		(drill 0.3)
-		(layers "F.Cu" "B.Cu")
-		(free yes)
-		(net 3)
-	)
-	(via
 		(at 199.471428 108.1)
 		(size 0.6)
@@
 	)
 	(via
-		(at 198.2 42.4)
-		(size 0.6)
-		(drill 0.3)
-		(layers "F.Cu" "B.Cu")
-		(free yes)
-		(net 3)
-	)
-	(via
 		(at 174.142857 106.4)
 		(size 0.6)
@@
 	)
 	(via
-		(at 185.214286 42.1)
-		(size 0.6)
-		(drill 0.3)
-		(layers "F.Cu" "B.Cu")
-		(free yes)
-		(net 3)
-	)
-	(via
 		(at 184.2 87)
 		(size 0.6)
@@
 	)
 	(via
-		(at 198.2 37.9)
-		(size 0.6)
-		(drill 0.3)
-		(layers "F.Cu" "B.Cu")
-		(free yes)
-		(net 3)
-	)
-	(via
 		(at 161.7 65.7)
 		(size 0.6)
@@
 	)
 	(via
-		(at 198.2 40.9)
-		(size 0.6)
-		(drill 0.3)
-		(layers "F.Cu" "B.Cu")
-		(free yes)
-		(net 3)
-	)
-	(via
 		(at 185.171429 37.5)
 		(size 0.6)
@@
 	)
 	(via
-		(at 176.728571 42.1)
-		(size 0.6)
-		(drill 0.3)
-		(layers "F.Cu" "B.Cu")
-		(free yes)
-		(net 3)
-	)
-	(via
 		(at 161.7 64.2)
 		(size 0.6)
@@
 	)
 	(via
-		(at 173.9 42.1)
-		(size 0.6)
-		(drill 0.3)
-		(layers "F.Cu" "B.Cu")
-		(free yes)
-		(net 3)
-	)
-	(via
 		(at 174.142857 107.9)
 		(size 0.6)
@@
 	)
 	(via
-		(at 168.2 41.9)
-		(size 0.6)
-		(drill 0.3)
-		(layers "F.Cu" "B.Cu")
-		(free yes)
-		(net 3)
-	)
-	(via
 		(at 161.671429 73.3)
 		(size 0.6)
@@
 	)
 	(via
-		(at 165.757143 44.9)
-		(size 0.6)
-		(drill 0.3)
-		(layers "F.Cu" "B.Cu")
-		(free yes)
-		(net 3)
-	)
-	(via
 		(at 167.328572 76.3)
 		(size 0.6)
@@
 	)
 	(via
-		(at 179.557143 42.1)
-		(size 0.6)
-		(drill 0.3)
-		(layers "F.Cu" "B.Cu")
-		(free yes)
-		(net 3)
-	)
-	(via
 		(at 164.5 79.3)
 		(size 0.6)
@@
 	)
 	(via
-		(at 168.2 43.4)
-		(size 0.6)
-		(drill 0.3)
-		(layers "F.Cu" "B.Cu")
-		(free yes)
-		(net 3)
-	)
-	(via
 		(at 195.328572 48.5)
 		(size 0.6)
@@
 	)
 	(via
-		(at 162.928572 46.4)
-		(size 0.6)
-		(drill 0.3)
-		(layers "F.Cu" "B.Cu")
-		(free yes)
-		(net 3)
-	)
-	(via
 		(at 210 87.2)
 		(size 0.6)
@@
 	)
 	(via
-		(at 198.2 43.9)
-		(size 0.6)
-		(drill 0.3)
-		(layers "F.Cu" "B.Cu")
-		(free yes)
-		(net 3)
-	)
-	(via
 		(at 192.5 54.5)
 		(size 0.6)
@@
 	)
 	(via
-		(at 182.385714 42.1)
-		(size 0.6)
-		(drill 0.3)
-		(layers "F.Cu" "B.Cu")
-		(free yes)
-		(net 3)
-	)
-	(via
 		(at 195.328572 60.5)
 		(size 0.6)
@@
 	)
 	(via
-		(at 198.2 39.4)
-		(size 0.6)
-		(drill 0.3)
-		(layers "F.Cu" "B.Cu")
-		(free yes)
-		(net 3)
-	)
-	(via
-		(at 188.042857 43.6)
-		(size 0.6)
-		(drill 0.3)
-		(layers "F.Cu" "B.Cu")
-		(free yes)
-		(net 3)
-	)
-	(via
 		(at 184.6 90.8)
 		(size 0.6)
@@
 		(size 0.6)
 		(drill 0.3)
-		(layers "F.Cu" "B.Cu")
-		(free yes)
-		(net 3)
-	)
-	(via
-		(at 188.042857 42.1)
-		(size 0.6)
-		(drill 0.3)

Commit message: layout done
Parts:
- removed H2: MountingHole_Pad, MountingHole:MountingHole_3.2mm_M3_Pad_TopBottom
- added 12V_SNS: 12V_Sense, TestPoint:TestPoint_Keystone_5000-5004_Miniature, F.Cu at (175.3, 92.7)
- added G***: LOGO, LOGO, F.Cu at (156.3, 84.8)
- added G***: LOGO, LOGO, F.Cu at (156.3, 87.8)
- added G***: LOGO, LOGO, F.Cu at (156.3, 82.2)
- added G***: LOGO, UTSVT_Logos:UTSVT_Logo_Symbol, B.Cu at (191.3, 50.0)
- added G***: LOGO, UTSVT_Logos:Hallock_Image_Tiny, B.Cu at (191.0, 59.9)
- added HSS_EN: TP_EN, TestPoint:TestPoint_Keystone_5000-5004_Miniature, F.Cu at (187.4, 96.3)
- added HSS_FAULT: TP_ST, TestPoint:TestPoint_Keystone_5000-5004_Miniature, F.Cu at (192.1, 96.3)
- added TP4: TP_PG, TestPoint:TestPoint_Keystone_5000-5004_Miniature, F.Cu at (202.0, 72.5)
- 24V1, TP_1, TP_2: footprint TestPoint:TestPoint_Pad_1.0x1.0mm -> TestPoint:TestPoint_Keystone_5000-5004_Miniature
- 3V3: renamed from 3V1; footprint TestPoint:TestPoint_Pad_1.0x1.0mm -> TestPoint:TestPoint_Keystone_5000-5004_Miniature
- BUCK_OUT: renamed from BUCK_OUT1; footprint TestPoint:TestPoint_Pad_1.0x1.0mm -> TestPoint:TestPoint_Keystone_5000-5004_Miniature
- C18: footprint Capacitor_SMD:C_0603_1608Metric_Pad1.08x0.95mm_HandSolder -> Capacitor_SMD:C_0805_2012Metric_Pad1.18x1.45mm_HandSolder
- F1: value 10A -> Fuse_3568; footprint Moco:FUSE_3568 -> UTSVT_Connectors:FUSE_3568
- FAULT: renamed from Fault1; footprint TestPoint:TestPoint_Pad_1.0x1.0mm -> TestPoint:TestPoint_Keystone_5000-5004_Miniature
- GND: renamed from TP1; footprint TestPoint:TestPoint_Pad_1.0x1.0mm -> TestPoint:TestPoint_Keystone_5000-5004_Miniature
- I_MOTOR: renamed from D_C1; footprint TestPoint:TestPoint_Pad_1.0x1.0mm -> TestPoint:TestPoint_Keystone_5000-5004_Miniature
- PP_OUT: renamed from 12V1; footprint TestPoint:TestPoint_Pad_1.0x1.0mm -> TestPoint:TestPoint_Keystone_5000-5004_Miniature
- PWM_A: renamed from PWM_A1; footprint TestPoint:TestPoint_Pad_1.0x1.0mm -> TestPoint:TestPoint_Keystone_5000-5004_Miniature
- PWM_B: renamed from PWM_B1; footprint TestPoint:TestPoint_Pad_1.0x1.0mm -> TestPoint:TestPoint_Keystone_5000-5004_Miniature
- STATUS: renamed from Message1; footprint TestPoint:TestPoint_Pad_1.0x1.0mm -> TestPoint:TestPoint_Keystone_5000-5004_Miniature
- SW_OC: renamed from OVC1; footprint TestPoint:TestPoint_Pad_1.0x1.0mm -> TestPoint:TestPoint_Keystone_5000-5004_Miniature
- moved C13 12.0 mm to (172.4, 67.7)
- moved C16 12.0 mm to (172.4, 69.2)
- moved R30 9.30 mm to (171.1, 56.9)
- moved C15 6.17 mm to (172.4, 64.7)
- moved C14 6.17 mm to (172.4, 66.2)
- moved C11 4.72 mm to (176.9, 71.0), turned to 0 degrees
- moved L1 4.15 mm to (177.4, 67.4), turned to 0 degrees
- moved C18 3.61 mm to (191.7, 79.5)
- moved C17 3.39 mm to (189.8, 79.2)
- moved R17 2.26 mm to (172.4, 63.1)
- moved TP_2 2.04 mm to (178.6, 96.3)
- moved LED7 1.99 mm to (178.6, 93.8)
- moved R8 1.99 mm to (178.6, 92.2)
- moved TP_1 1.80 mm to (183.2, 96.3)
- moved R28 1.76 mm to (192.1, 93.9)
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- renumbered LED6 to PB0, TACH_A1 to TACH_A, TACH_B1 to TACH_B
Routing:
- net /12V_BUS: track 3.37 -> 28.3 mm
- net +12V: track 0.00 -> 21.1 mm
- net /Power12V/RPP_EN: track 3.69 -> 15.6 mm
- net /12V_SENSE: track 28.7 -> 37.8 mm, vias 2 -> 3
- net /PSOM_PWR: track 3.45 -> 11.3 mm, vias 2 -> 1
- net /CAN_H: track 148.1 -> 154.3 mm, vias 1 -> 2
- net /EN: track 21.0 -> 26.7 mm
- net /CAN_L: track 134.4 -> 139.9 mm, vias 1 -> 2
- net Net-(U1-BOOT): track 2.67 -> 8.01 mm, vias 0 -> 2
- net Net-(U1-FB): track 0.00 -> 5.13 mm
- net Net-(U1-PG): track 14.6 -> 19.3 mm
- net /FAN_B_TACHO: track 25.0 -> 29.4 mm
- net /M_FAULT: track 40.6 -> 43.8 mm
- net Net-(D3-K): track 18.5 -> 21.7 mm
- net +3V3: track 84.8 -> 87.4 mm
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- removed copper zone on F.Cu, net /Power12V/RPP_EN
- removed copper zone on F.Cu, net Net-(U1-FB)
Other:
- board size 59.1 x 75.7 mm -> 62.8 x 79.5 mm
- board text added: "59.2"
- board text added: "75.9"
- board text added: "LATCH PB15"
- board text added: "LHRS PS-Moco Interface RevB 2026 Jennifer Li"
- board text added: "PA12"
- board text added: "PA2"
- board text added: "PA4"
- board text added: "PA5"
- board text added: "PA6"
- board text added: "PB10"
- board text added: "PB12"
- board text added: "PB14"
- board text added: "PB6"
- board text added: "PB7"
- board text added: "Spot reserved for Richard"
- board text removed: "LHRS RevB Jennifer Li 2026"
- board text removed: "Moco Interface LHR Rev A 2025 Jennifer Li"

Commit message: layout changes made
Parts:
- moved JP1 2.03 mm to (200.7, 105.2)
- moved R4 2.00 mm to (200.7, 107.8)
- moved H1 1.50 mm to (206.9, 92.3)
- moved R11 1.43 mm to (171.2, 86.1)
- moved GND 0.45 mm to (201.0, 96.3)
- moved G*** 0.05 mm to (156.3, 84.9)
- renumbered 24V1 to 24V, TP4 to BUCK_PG
Routing:
- net /CAN_H: track 154.3 -> 158.0 mm
- net /CAN_L: track 139.9 -> 142.0 mm
- net /PWM_FAN_A: track 23.8 -> 24.5 mm
- net GND: vias 335 -> 332
