File: Hardware/KiCad/BuckConverter.kicad_sch (KiCad schematic)
At the start: 18 parts, among them U1 LMR33630ADDA

Commit message: standardized some lcsc
Parts:
- D15: LCSC C7371904 -> C84263
Changed lines of the file:
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@@
 			)
 		)
-		(property "LCSC" "C7371904"
+		(property "LCSC" "C84263"
 			(at 130.81 127 90)
 			(effects
